Commit message: added simplified IRB_6400 URDF

File: models/plane.urdf (robot description, URDF)
Before this commit: robot plane, 1 links, 0 joints
Links:
- link planeLink: geometry collision box size=3 3 1; visual mesh filename=plane.obj scale=1 1 1

Commit message: fixed falling through plane bug

File: models/plane.urdf (robot description, URDF)
Before this commit: robot plane, 1 links, 0 joints
Links:
- link planeLink: geometry collision box size=15 15 1; visual mesh filename=plane.obj scale=1 1 1

File: models/table.urdf (robot description, URDF)
Before this commit: robot table, 5 links, 4 joints
Links:
- link leg_1: mass 100 -> 1
- link leg_2: mass 100 -> 1
- link leg_3: mass 100 -> 1
- link leg_4: mass 100 -> 1
- link tabletop: mass 100 -> 1
Joints:
- joint joint_1: origin xyz=0.25 0.25 -0.15 rpy=0 0 0 -> xyz=0.20 0.20 -0.15 rpy=0 0 0
- joint joint_2: origin xyz=-0.25 0.25 -0.15 rpy=0 0 0 -> xyz=-0.20 0.20 -0.15 rpy=0 0 0
- joint joint_3: origin xyz=0.25 -0.25 -0.15 rpy=0 0 0 -> xyz=0.20 -0.20 -0.15 rpy=0 0 0
- joint joint_4: origin xyz=-0.25 -0.25 -0.15 rpy=0 0 0 -> xyz=-0.20 -0.20 -0.15 rpy=0 0 0
