Commit message: fixed axis of rotation for wrist axes

File: models/IRB_6400.urdf (robot description, URDF)
Before this commit: robot IRB_6400, 7 links, 6 joints
Joints:
- joint joint_4: axis 1 0 0 -> 0 0 1
- joint joint_5: axis 0 1 0 -> 0 0 1
- joint joint_6: axis 1 0 0 -> 0 0 1

Commit message: fix inertial issues

File: models/IRB_6400.urdf (robot description, URDF)
Before this commit: robot IRB_6400, 7 links, 6 joints
Links:
- link base: mass None -> 100
- link link_1: mass None -> 1
- link link_2: mass None -> 1
- link link_3: mass None -> 1
- link link_4: mass None -> 1
- link link_5: mass None -> 1
- link link_6: mass None -> 1

Commit message: update todo and urdf

File: models/IRB_6400.urdf (robot description, URDF)
Before this commit: robot IRB_6400, 7 links, 6 joints
Links:
- added link end_effector, mass 0.1; collision sphere radius=0.05; visual sphere radius=0.05
- link link_5: geometry collision cylinder length=0 radius=0.1; visual cylinder length=0 radius=0.1
- link link_6: geometry collision cylinder length=0 radius=0.1; visual cylinder length=0 radius=0.1
Joints:
- added joint joint_7: type fixed, parent link_6, child end_effector, origin xyz=0 0 -0.1 rpy=0 0 0
- joint joint_1: limit lower=0.0 upper=6.28 effort=1000.0 velocity=0.5 -> lower=-3.14 upper=3.14 effort=1000.0 velocity=0.5
- joint joint_2: limit lower=0.0 upper=6.28 effort=1000.0 velocity=0.5 -> lower=-1.2 upper=1.4 effort=1000.0 velocity=0.5
- joint joint_3: limit lower=0.0 upper=6.28 effort=1000.0 velocity=0.5 -> lower=-0.48 upper=1.91 effort=1000.0 velocity=0.5
- joint joint_4: limit lower=0.0 upper=6.28 effort=1000.0 velocity=0.5 -> lower=-5.2 upper=5.2 effort=1000.0 velocity=0.5
- joint joint_5: limit lower=0.0 upper=6.28 effort=1000.0 velocity=0.5 -> lower=-2.09 upper=2.09 effort=1000.0 velocity=0.5
- joint joint_6: limit lower=0.0 upper=6.28 effort=1000.0 velocity=0.5 -> lower=-5.2 upper=5.2 effort=1000.0 velocity=0.5

Commit message: -Added damping/friction to urdf model -Improved starting/end position

File: models/IRB_6400.urdf (robot description, URDF)
Before this commit: robot IRB_6400, 8 links, 7 joints
Joints:
- joint joint_1: limit lower=-3.14 upper=3.14 effort=1000.0 velocity=0.5 -> lower=-3.14 upper=3.14 effort=10.0 velocity=0.01
- joint joint_2: limit lower=-1.2 upper=1.4 effort=1000.0 velocity=0.5 -> lower=-1.2 upper=1.4 effort=10.0 velocity=0.01
- joint joint_3: limit lower=-0.48 upper=1.91 effort=1000.0 velocity=0.5 -> lower=-0.48 upper=1.91 effort=10.0 velocity=0.01
- joint joint_4: limit lower=-5.2 upper=5.2 effort=1000.0 velocity=0.5 -> lower=-5.2 upper=5.2 effort=10.0 velocity=0.01
- joint joint_5: limit lower=-2.09 upper=2.09 effort=1000.0 velocity=0.5 -> lower=-2.09 upper=2.09 effort=10.0 velocity=0.01
- joint joint_6: limit lower=-5.2 upper=5.2 effort=1000.0 velocity=0.5 -> lower=-5.2 upper=5.2 effort=10.0 velocity=0.01

Commit message: simulation is now bugless

File: models/IRB_6400.urdf (robot description, URDF)
Before this commit: robot IRB_6400, 8 links, 7 joints
Joints:
- joint joint_1: limit lower=-3.14 upper=3.14 effort=10.0 velocity=0.01 -> lower=-3.14 upper=3.14 effort=100.0 velocity=0.01
- joint joint_2: limit lower=-1.2 upper=1.4 effort=10.0 velocity=0.01 -> lower=-1.2 upper=1.4 effort=100.0 velocity=0.01
- joint joint_3: limit lower=-0.48 upper=1.91 effort=10.0 velocity=0.01 -> lower=-0.48 upper=1.91 effort=100.0 velocity=0.01
- joint joint_4: limit lower=-5.2 upper=5.2 effort=10.0 velocity=0.01 -> lower=-5.2 upper=5.2 effort=100.0 velocity=0.01
- joint joint_5: limit lower=-2.09 upper=2.09 effort=10.0 velocity=0.01 -> lower=-2.09 upper=2.09 effort=100.0 velocity=0.01
- joint joint_6: limit lower=-5.2 upper=5.2 effort=10.0 velocity=0.01 -> lower=-5.2 upper=5.2 effort=100.0 velocity=0.01

File: models/block.urdf (robot description, URDF)
Before this commit: robot block, 1 links, 0 joints
Links:
- link block: geometry collision box size=2 2 0.4; visual box size=2 2 0.4
